Commit message: more changes

File: urdf/combined.urdf.xacro (robot description, xacro)
@@ -13,5 +13,5 @@
       <origin xyz="0.3576 0.4515 -0.335" rpy="1.5708 0 -1.5708"/>
       <geometry>
-        <mesh filename="package://feeding_deployment/urdf/meshes/feeding_vention_modification.STL"
+        <mesh filename="package://feeding_deployment/urdf/meshes/feeding_vention_modification_decimated.STL"
               scale="0.001 0.001 0.001"/>
       </geometry>
